File: panel/back_panel/back_panel.kicad_pcb (KiCad board)
At the start: 2 copper layers, 100 x 100 mm, 0 parts

Commit message: add panel stuff
Routing:
- net (no net): track 7.67 -> 0.00 mm
Other:
- outline, holes or cut-outs redrawn
Changed lines of the file:
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@@
   (net 0 "")
   (gr_line (start 181.65 144.75) (end 81.65 144.75) (layer "Edge.Cuts") (width 0.15))
-  (gr_circle (center 178.138276 48.238276) (end 179.838276 48.038276) (layer "Edge.Cuts") (width 0.1) (fill none))
-  (gr_circle (center 85.15 141.261724) (end 86.85 141.061724) (layer "Edge.Cuts") (width 0.1) (fill none))
+  (gr_circle (center 178.15 48.25) (end 179.85 48.05) (layer "Edge.Cuts") (width 0.1) (fill none))
+  (gr_circle (center 85.15 141.25) (end 86.85 141.05) (layer "Edge.Cuts") (width 0.1) (fill none))
   (gr_line (start 81.65 44.75) (end 181.65 44.75) (layer "Edge.Cuts") (width 0.15))
   (gr_circle (center 85.15 48.25) (end 86.85 48.05) (layer "Edge.Cuts") (width 0.1) (fill none))
   (gr_line (start 181.65 44.75) (end 181.65 144.75) (layer "Edge.Cuts") (width 0.15))
-  (gr_circle (center 178.138276 141.25) (end 179.838276 141.05) (layer "Edge.Cuts") (width 0.1) (fill none))
+  (gr_circle (center 178.15 141.2) (end 179.85 141) (layer "Edge.Cuts") (width 0.1) (fill none))
   (gr_line (start 81.65 144.75) (end 81.65 44.75) (layer "Edge.Cuts") (width 0.15))
   (gr_text "JLCJLCJLCJLC" (at 171.95 143.55) (layer "B.SilkS")
     (effects (font (size 1 1) (thickness 0.15)) (justify mirror))
   )
-  (segment (start 175.4 142) (end 167.8 142) (width 0.25) (layer "B.Cu") (net 0))
-  (segment (start 167.8 142) (end 167.75 142.05) (width 0.25) (layer "B.Cu") (net 0))
 )
