File: panel/eurorack_panel/eurorack_panel.kicad_pcb (KiCad board)
At the start: 2 copper layers, 101.6 x 128.6 mm, 2 parts

Commit message: some panel stuff
Routing:
- net (no net): track 0.00 -> 7.90 mm
Other:
- outline, holes or cut-outs redrawn
- board text added: "cyberboy666 & ichi raramuri recurBOY panel for v0_7_1 mk_iii"
- board text removed: "cyberboy666 & ichi raramuri recurBOY panel for v0_7_1 mk_ii"
